Commit message: first commit in this branch

File: config/gazebo_mycobot_pro.urdf (robot description, URDF)
Before this commit: robot mycobot_pro, 8 links, 7 joints
Links:
- added link magsensor, mass 0.2; collision box size=0.01 0.002 0.01; visual box size=0.01 0.01 0.002
Joints:
- added joint link6_to_magsensor: type fixed, parent link6, child magsensor, origin xyz=-0.03 -0.0 0.001 rpy=0 0 -1.5708 

Commit message: change urdf

File: config/gazebo_mycobot_pro.urdf (robot description, URDF)
Before this commit: robot mycobot_pro, 9 links, 8 joints
Joints:
- joint arm_joint_0: limit lower=-3.14 upper=3.14159 effort=100.0 velocity=5 -> lower=-2.96706 upper=2.96706 effort=100.0 velocity=5
- joint arm_joint_1: limit lower=-3.14 upper=3.14159 effort=100.0 velocity=5 -> lower=-2.7925268 upper=2.7925268 effort=100.0 velocity=5
- joint arm_joint_2: limit lower=-3.14 upper=3.14159 effort=100.0 velocity=5 -> lower=-2.7925268 upper=2.7925268 effort=100.0 velocity=5
- joint arm_joint_3: limit lower=-3.14 upper=3.14159 effort=100.0 velocity=5 -> lower=-2.7925268 upper=2.7925268 effort=100.0 velocity=5
- joint arm_joint_4: limit lower=-3.14 upper=3.14159 effort=100.0 velocity=5 -> lower=-2.96706 upper=2.96706 effort=100.0 velocity=5
- joint arm_joint_5: limit lower=-3.14 upper=3.14159 effort=100.0 velocity=5 -> lower=-3.054326 upper=3.054326 effort=100.0 velocity=5
- joint link6_to_magsensor: origin xyz=-0.03 -0.0 0.001 rpy=0 0 -1.5708  -> xyz=-0.025 -0.0 0.001 rpy=0 0 -1.5708 

Commit message: change sensor position

File: config/gazebo_mycobot_pro.urdf (robot description, URDF)
Before this commit: robot mycobot_pro, 9 links, 8 joints
Joints:
- joint link6_to_magsensor: origin xyz=-0.025 -0.0 0.001 rpy=0 0 -1.5708  -> xyz=-0.0 -0.005 0.0 rpy=0 0 3.141592

Commit message: change sensor position

File: config/gazebo_mycobot_pro.urdf (robot description, URDF)
Before this commit: robot mycobot_pro, 9 links, 8 joints
Joints:
- joint link6_to_magsensor: origin xyz=-0.0 -0.005 0.0 rpy=0 0 3.141592 -> xyz=-0.0 -0.005 -0.008 rpy=0 0 3.141592

Commit message: change sensor position

File: config/gazebo_mycobot_pro.urdf (robot description, URDF)
Before this commit: robot mycobot_pro, 9 links, 8 joints
Joints:
- joint link6_to_magsensor: origin xyz=-0.0 -0.005 -0.008 rpy=0 0 3.141592 -> xyz=-0.0 -0.00 -0.006 rpy=0 0 3.141592
